Commit message: removed wheels, step 2 done

File: mobile_robot_description/xacro/robot.xacro (robot description, xacro)
@@ -1,22 +1,4 @@
 <?xml version="1.0"?>
 <robot xmlns:xacro="http://www.ros.org/wiki/xacro"  name="mobile_robot">
-  <xacro:macro name="wheel">
-    <visual>
-      <origin xyz="0.02 0 0" rpy="0 0 ${pi/2}"/>
-      <geometry>
-        <box size="0.6 0.4 0.10"/>
-      </geometry>
-    </visual>
-    <inertial>
-      <mass value="0.5"/>
-      <inertia ixx="0.0" ixy="0.0" ixz="0.0" iyy="0.000001" iyz="0.0" izz="0.0"/>
-    </inertial>
-    <collision>
-      <origin xyz="0.027 0 0.0" rpy="0 ${pi/2} 0"/>
-      <geometry>
-         <cylinder length="0.045" radius="0.08"/>
-      </geometry>
-    </collision>
-  </xacro:macro>
   <link name="base_link">
     <visual>

Commit message: added wheel

File: mobile_robot_description/xacro/robot.xacro (robot description, xacro)
@@ -1,4 +1,26 @@
 <?xml version="1.0"?>
 <robot xmlns:xacro="http://www.ros.org/wiki/xacro"  name="mobile_robot">
+  <xacro:macro name="wheel" params="name x y">
+    <link name="${name}">
+      <visual>
+        <origin xyz="0 0 0" rpy="${pi/2} 0 0"/>
+        <geometry>
+          <cylinder length="0.04" radius="0.1"/>
+        </geometry>
+      </visual>
+      <collision>
+        <origin xyz="0 0 0" rpy="${pi/2} 0 0"/>
+        <geometry>
+           <cylinder length="0.04" radius="0.1"/>
+        </geometry>
+      </collision>
+    </link>
+    <joint name="base_link_${name}" type="continuous">
+      <origin xyz="${y*0.25} ${x*0.25} 0" rpy="0 0 ${(x-1)* pi/2}"/>
+       <axis rpy="0 0 0" xyz="0 1 0"/>
+      <parent link="base_link"/>
+      <child link="${name}"/>
+    </joint>
+  </xacro:macro>
   <link name="base_link">
     <visual>
@@ -18,3 +40,38 @@
     </collision>
   </link>
+  <xacro:wheel name="wh_left_back" x="1" y="-1"/>
+  <xacro:wheel name="wh_right_back" x="-1" y="-1"/>
+  <xacro:wheel name="wh_left_front" x="1" y="1"/>
+  <xacro:wheel name="wh_right_front" x="-1" y="1"/>
+  <!-- ===================== References ===================== -->
+  <link name="x">
+    <visual>
+      <geometry>
+        <sphere radius="0.1"/>
+      </geometry>
+      <material name="x">
+        <color rgba="1.0 0.0 0.0 0.3"/>
+      </material>
+    </visual>
+  </link>
+  <joint name="base_link_x" type="fixed">
+    <origin xyz="1.0 0 0" rpy="0 0 0"/>
+    <parent link="base_link"/>
+    <child link="x"/>
+  </joint>
+  <link name="y">
+    <visual>
+      <geometry>
+        <sphere radius="0.1"/>
+      </geometry>
+      <material name="y">
+        <color rgba="0.0 1.0 0.0 0.3"/>
+      </material>
+    </visual>
+  </link>
+  <joint name="base_link_y" type="fixed">
+    <origin xyz="0 1 0" rpy="0 0 0"/>
+    <parent link="base_link"/>
+    <child link="y"/>
+  </joint>
 </robot>

Commit message: after gazebo, step 4

File: mobile_robot_description/xacro/robot.xacro (robot description, xacro)
@@ -1,4 +1,10 @@
 <?xml version="1.0"?>
 <robot xmlns:xacro="http://www.ros.org/wiki/xacro"  name="mobile_robot">
+  <xacro:macro name="default_inertial" params="mass">
+    <inertial>
+      <mass value="${mass}" />
+      <inertia ixx="1.0" ixy="0.0" ixz="0.0" iyy="1.0" iyz="0.0" izz="1.0" />
+    </inertial>
+  </xacro:macro>
   <xacro:macro name="wheel" params="name x y">
     <link name="${name}">
@@ -15,4 +21,5 @@
         </geometry>
       </collision>
+      <xacro:default_inertial mass="0.6"/>
     </link>
     <joint name="base_link_${name}" type="continuous">
@@ -39,4 +46,5 @@
       </geometry>
     </collision>
+    <xacro:default_inertial mass="6"/>
   </link>
   <xacro:wheel name="wh_left_back" x="1" y="-1"/>
@@ -45,4 +53,5 @@
   <xacro:wheel name="wh_right_front" x="-1" y="1"/>
   <!-- ===================== References ===================== -->
+  <!--
   <link name="x">
     <visual>
@@ -75,3 +84,23 @@
     <child link="y"/>
   </joint>
+  -->
+  <!-- =================== Gazebo ==================== -->
+  <gazebo>
+    <plugin name="gazebo_ros_control" filename="libgazebo_ros_control.so">
+      <robotNamespace>/</robotNamespace>
+    </plugin>
+  </gazebo>
+  <!-- <plugin name="differential_drive_controller" filename="libgazebo_ros_diff_drive.so">
+    <alwaysOn>true</alwaysOn>
+    <updateRate>20</updateRate>
+    <leftJoint>base_link_wh_left_back</leftJoint>
+    <rightJoint>base_link_wh_right_back</rightJoint>
+    <wheelSeparation>0.5</wheelSeparation>
+    <wheelDiameter>0.1</wheelDiameter>
+    <torque>20</torque>
+    <commandTopic>cmd_vel</commandTopic>
+    <odometryTopic>odom</odometryTopic>
+    <odometryFrame>odom</odometryFrame>
+    <robotBaseFrame>base_footprint</robotBaseFrame>
+  </plugin> -->
 </robot>

Commit message: step 2 done in gazebo

File: mobile_robot_description/xacro/robot.xacro (robot description, xacro)
@@ -29,4 +29,20 @@
       <child link="${name}"/>
     </joint>
+    <gazebo reference="base_link_${name}_wheel">
+      <mu1 value="200.0"/>
+      <mu2 value="100.0"/>
+      <kp value="10000000.0" />
+      <kd value="1.0" />
+      <material>Gazebo/Grey</material>
+    </gazebo>
+    <transmission name="base_link_${name}_wheel_trans">
+      <type>transmission_interface/SimpleTransmission</type>
+      <actuator name="base_link_${name}_wheel_motor">
+        <mechanicalReduction>1</mechanicalReduction>
+      </actuator>
+      <joint name="base_link_${name}">
+        <hardwareInterface>hardware_interface/VelocityJointInterface</hardwareInterface>
+      </joint>
+    </transmission>
   </xacro:macro>
   <link name="base_link">

Commit message: diffdrive working

File: mobile_robot_description/xacro/robot.xacro (robot description, xacro)
@@ -24,5 +24,5 @@
     </link>
     <joint name="base_link_${name}" type="continuous">
-      <origin xyz="${y*0.25} ${x*0.25} 0" rpy="0 0 ${(x-1)* pi/2}"/>
+      <origin xyz="${y*0.25} ${x*0.25} 0" rpy="0 0 0"/>
        <axis rpy="0 0 0" xyz="0 1 0"/>
       <parent link="base_link"/>
@@ -30,7 +30,7 @@
     </joint>
     <gazebo reference="base_link_${name}_wheel">
-      <mu1 value="200.0"/>
-      <mu2 value="100.0"/>
-      <kp value="10000000.0" />
+      <mu1 value="20.0"/>
+      <mu2 value="10.0"/>
+      <kp value="1000.0" />
       <kd value="1.0" />
       <material>Gazebo/Grey</material>

Commit message: section 1 part 2

File: mobile_robot_description/xacro/robot.xacro (robot description, xacro)
@@ -1,10 +1,4 @@
 <?xml version="1.0"?>
-<robot xmlns:xacro="http://www.ros.org/wiki/xacro"  name="mobile_robot">
-  <xacro:macro name="default_inertial" params="mass">
-    <inertial>
-      <mass value="${mass}" />
-      <inertia ixx="1.0" ixy="0.0" ixz="0.0" iyy="1.0" iyz="0.0" izz="1.0" />
-    </inertial>
-  </xacro:macro>
+<robot xmlns:xacro="http://www.ros.org/wiki/xacro" name="mobile_robot">
   <xacro:macro name="wheel" params="name x y">
     <link name="${name}">
@@ -18,31 +12,14 @@
         <origin xyz="0 0 0" rpy="${pi/2} 0 0"/>
         <geometry>
-           <cylinder length="0.04" radius="0.1"/>
+          <cylinder length="0.04" radius="0.1"/>
         </geometry>
       </collision>
-      <xacro:default_inertial mass="0.6"/>
     </link>
     <joint name="base_link_${name}" type="continuous">
       <origin xyz="${y*0.25} ${x*0.25} 0" rpy="0 0 0"/>
-       <axis rpy="0 0 0" xyz="0 1 0"/>
+      <axis rpy="0 0 0" xyz="0 1 0"/>
       <parent link="base_link"/>
       <child link="${name}"/>
     </joint>
-    <gazebo reference="base_link_${name}_wheel">
-      <mu1 value="20.0"/>
-      <mu2 value="10.0"/>
-      <kp value="1000.0" />
-      <kd value="1.0" />
-      <material>Gazebo/Grey</material>
-    </gazebo>
-    <transmission name="base_link_${name}_wheel_trans">
-      <type>transmission_interface/SimpleTransmission</type>
-      <actuator name="base_link_${name}_wheel_motor">
-        <mechanicalReduction>1</mechanicalReduction>
-      </actuator>
-      <joint name="base_link_${name}">
-        <hardwareInterface>hardware_interface/VelocityJointInterface</hardwareInterface>
-      </joint>
-    </transmission>
   </xacro:macro>
   <link name="base_link">
@@ -62,5 +39,4 @@
       </geometry>
     </collision>
-    <xacro:default_inertial mass="6"/>
   </link>
   <xacro:wheel name="wh_left_back" x="1" y="-1"/>
@@ -68,55 +44,3 @@
   <xacro:wheel name="wh_left_front" x="1" y="1"/>
   <xacro:wheel name="wh_right_front" x="-1" y="1"/>
-  <!-- ===================== References ===================== -->
-  <!--
-  <link name="x">
-    <visual>
-      <geometry>
-        <sphere radius="0.1"/>
-      </geometry>
-      <material name="x">
-        <color rgba="1.0 0.0 0.0 0.3"/>
-      </material>
-    </visual>
-  </link>
-  <joint name="base_link_x" type="fixed">
-    <origin xyz="1.0 0 0" rpy="0 0 0"/>
-    <parent link="base_link"/>
-    <child link="x"/>
-  </joint>
-  <link name="y">
-    <visual>
-      <geometry>
-        <sphere radius="0.1"/>
-      </geometry>
-      <material name="y">
-        <color rgba="0.0 1.0 0.0 0.3"/>
-      </material>
-    </visual>
-  </link>
-  <joint name="base_link_y" type="fixed">
-    <origin xyz="0 1 0" rpy="0 0 0"/>
-    <parent link="base_link"/>
-    <child link="y"/>
-  </joint>
-  -->
-  <!-- =================== Gazebo ==================== -->
-  <gazebo>
-    <plugin name="gazebo_ros_control" filename="libgazebo_ros_control.so">
-      <robotNamespace>/</robotNamespace>
-    </plugin>
-  </gazebo>
-  <!-- <plugin name="differential_drive_controller" filename="libgazebo_ros_diff_drive.so">
-    <alwaysOn>true</alwaysOn>
-    <updateRate>20</updateRate>
-    <leftJoint>base_link_wh_left_back</leftJoint>
-    <rightJoint>base_link_wh_right_back</rightJoint>
-    <wheelSeparation>0.5</wheelSeparation>
-    <wheelDiameter>0.1</wheelDiameter>
-    <torque>20</torque>
-    <commandTopic>cmd_vel</commandTopic>
-    <odometryTopic>odom</odometryTopic>
-    <odometryFrame>odom</odometryFrame>
-    <robotBaseFrame>base_footprint</robotBaseFrame>
-  </plugin> -->
 </robot>

Commit message: Section 1 part 3

File: mobile_robot_description/xacro/robot.xacro (robot description, xacro)
@@ -1,4 +1,16 @@
 <?xml version="1.0"?>
 <robot xmlns:xacro="http://www.ros.org/wiki/xacro" name="mobile_robot">
+  <xacro:macro name="default_inertial" params="mass">
+    <inertial>
+      <mass value="${mass}"/>
+      <inertia ixx="1.0" ixy="0.0" ixz="0.0" iyy="1.0" iyz="0.0" izz="1.0"/>
+    </inertial>
+  </xacro:macro>
+  <xacro:macro name="default_inertial" params="mass">
+    <inertial>
+      <mass value="${mass}"/>
+      <inertia ixx="1.0" ixy="0.0" ixz="0.0" iyy="1.0" iyz="0.0" izz="1.0"/>
+    </inertial>
+  </xacro:macro>
   <xacro:macro name="wheel" params="name x y">
     <link name="${name}">
@@ -15,4 +27,5 @@
         </geometry>
       </collision>
+      <xacro:default_inertial mass="0.6"/>
     </link>
     <joint name="base_link_${name}" type="continuous">
@@ -39,4 +52,5 @@
       </geometry>
     </collision>
+    <xacro:default_inertial mass="6"/>
   </link>
   <xacro:wheel name="wh_left_back" x="1" y="-1"/>
@@ -44,3 +58,22 @@
   <xacro:wheel name="wh_left_front" x="1" y="1"/>
   <xacro:wheel name="wh_right_front" x="-1" y="1"/>
+  <!-- =================== Gazebo ==================== -->
+  <gazebo>
+    <plugin name="gazebo_ros_control" filename="libgazebo_ros_control.so">
+      <robotNamespace>/</robotNamespace>
+    </plugin>
+  </gazebo>
+  <plugin name="differential_drive_controller" filename="libgazebo_ros_diff_drive.so">
+    <alwaysOn>true</alwaysOn>
+    <updateRate>20</updateRate>
+    <leftJoint>base_link_wh_left_back</leftJoint>
+    <rightJoint>base_link_wh_right_back</rightJoint>
+    <wheelSeparation>0.5</wheelSeparation>
+    <wheelDiameter>0.1</wheelDiameter>
+    <torque>20</torque>
+    <commandTopic>cmd_vel</commandTopic>
+    <odometryTopic>odom</odometryTopic>
+    <odometryFrame>odom</odometryFrame>
+    <robotBaseFrame>base_footprint</robotBaseFrame>
+  </plugin>
 </robot>

Commit message: section 1 part 4

File: mobile_robot_description/xacro/robot.xacro (robot description, xacro)
@@ -35,4 +35,20 @@
       <child link="${name}"/>
     </joint>
+    <gazebo reference="base_link_${name}_wheel">
+      <mu1 value="200.0"/>
+      <mu2 value="100.0"/>
+      <kp value="10000000.0"/>
+      <kd value="1.0"/>
+      <material>Gazebo/Grey</material>
+    </gazebo>
+    <transmission name="base_link_${name}_wheel_trans">
+      <type>transmission_interface/SimpleTransmission</type>
+      <actuator name="base_link_${name}_wheel_motor">
+        <mechanicalReduction>1</mechanicalReduction>
+      </actuator>
+      <joint name="base_link_${name}">
+        <hardwareInterface>hardware_interface/VelocityJointInterface</hardwareInterface>
+      </joint>
+    </transmission>
   </xacro:macro>
   <link name="base_link">

Commit message: Section 2 part 1

File: mobile_robot_description/xacro/robot.xacro (robot description, xacro)
@@ -74,4 +74,28 @@
   <xacro:wheel name="wh_left_front" x="1" y="1"/>
   <xacro:wheel name="wh_right_front" x="-1" y="1"/>
+  <!-- =================== Kinect ==================== -->
+  <link name="kinect_link">
+    <visual>
+      <origin xyz="0 0 0" rpy="0 0 0"/>
+      <geometry>
+        <mesh filename="package://mobile_robot_description/meshes/kinect.stl" scale="0.01 0.01 0.01"/>
+      </geometry>
+      <material name="kinect">
+        <color rgba="1 0.9 0.9 1"/>
+      </material>
+    </visual>
+    <collision>
+      <origin xyz="0 0 0" rpy="0 0 0"/>
+      <geometry>
+        <box size="0.28 0.07 0.08"/>
+      </geometry>
+    </collision>
+    <xacro:default_inertial mass="0.2"/>
+  </link>
+  <joint name="base_link_kinect_link" type="fixed">
+    <origin xyz="0.265 0 0.087" rpy="0 0 ${pi/2}"/>
+    <parent link="base_link"/>
+    <child link="kinect_link"/>
+  </joint>
   <!-- =================== Gazebo ==================== -->
   <gazebo>

Commit message: Section 2 part 2

File: mobile_robot_description/xacro/robot.xacro (robot description, xacro)
@@ -35,11 +35,4 @@
       <child link="${name}"/>
     </joint>
-    <gazebo reference="base_link_${name}_wheel">
-      <mu1 value="200.0"/>
-      <mu2 value="100.0"/>
-      <kp value="10000000.0"/>
-      <kd value="1.0"/>
-      <material>Gazebo/Grey</material>
-    </gazebo>
     <transmission name="base_link_${name}_wheel_trans">
       <type>transmission_interface/SimpleTransmission</type>
@@ -68,5 +61,5 @@
       </geometry>
     </collision>
-    <xacro:default_inertial mass="6"/>
+    <xacro:default_inertial mass="20"/>
   </link>
   <xacro:wheel name="wh_left_back" x="1" y="-1"/>
@@ -98,4 +91,76 @@
     <child link="kinect_link"/>
   </joint>
+  <!-- =================== Gazebo - Kinect ==================== -->
+  <link name="gz_kinect_link">
+    <visual>
+      <origin xyz="0 0 0" rpy="0 0 0"/>
+      <geometry>
+        <sphere radius="0.05"/>
+      </geometry>
+      <material name="kinect">
+        <color rgba="1 0.9 0.9 1"/>
+      </material>
+    </visual>
+    <collision>
+      <origin xyz="0 0 0" rpy="0 0 0"/>
+      <geometry>
+        <sphere radius="0.05"/>
+      </geometry>
+    </collision>
+    <xacro:default_inertial mass="0.2"/>
+  </link>
+  <joint name="kinect_link_gz_kinect_link" type="fixed">
+    <origin xyz="0 0 0" rpy="0 0 -${pi/2}"/>
+    <parent link="kinect_link"/>
+    <child link="gz_kinect_link"/>
+  </joint>
+  <gazebo reference="gz_kinect_link">
+    <sensor type="depth" name="kinect">
+      <pose>0 0 0 0 0 0</pose>
+      <always_on>1</always_on>
+      <visualize>true</visualize>
+      <camera>
+        <horizontal_fov>1.047</horizontal_fov>
+        <image>
+          <width>640</width>
+          <height>480</height>
+          <format>R8G8B8</format>
+        </image>
+        <depth_camera></depth_camera>
+        <clip>
+          <near>0.1</near>
+          <far>100</far>
+        </clip>
+        <noise>
+          <type>gaussian</type>
+          <mean>0.0</mean>
+          <stddev>0.7</stddev>
+        </noise>
+      </camera>
+      <plugin name="camera_controller" filename="libgazebo_ros_openni_kinect.so">
+        <!-- <baseline>0.2</baseline> -->
+        <alwaysOn>true</alwaysOn>
+        <updateRate>10.0</updateRate>
+        <cameraName>kinect_sensor</cameraName>
+        <frameName>gz_kinect_link</frameName>
+        <imageTopicName>/mobile_robot/rgb/image_raw</imageTopicName>
+        <depthImageTopicName>/mobile_robot/depth/image_raw</depthImageTopicName>
+        <pointCloudTopicName>/mobile_robot/depth/points</pointCloudTopicName>
+        <cameraInfoTopicName>/mobile_robot/rgb/camera_info</cameraInfoTopicName>
+        <depthImageInfoTopicName>/mobile_robot/depth/camera_info</depthImageInfoTopicName>
+        <pointCloudCutoff>0.4</pointCloudCutoff>
+        <hackBaseline>0.07</hackBaseline>
+        <distortionK1>0.001</distortionK1>
+        <distortionK2>0.001</distortionK2>
+        <distortionK3>0.001</distortionK3>
+        <distortionT1>0.001</distortionT1>
+        <distortionT2>0.001</distortionT2>
+        <CxPrime>0</CxPrime>
+        <Cx>0</Cx>
+        <Cy>0</Cy>
+        <focalLength>0</focalLength>
+      </plugin>
+    </sensor>
+  </gazebo>
   <!-- =================== Gazebo ==================== -->
   <gazebo>
@@ -104,16 +169,3 @@
     </plugin>
   </gazebo>
-  <plugin name="differential_drive_controller" filename="libgazebo_ros_diff_drive.so">
-    <alwaysOn>true</alwaysOn>
-    <updateRate>20</updateRate>
-    <leftJoint>base_link_wh_left_back</leftJoint>
-    <rightJoint>base_link_wh_right_back</rightJoint>
-    <wheelSeparation>0.5</wheelSeparation>
-    <wheelDiameter>0.1</wheelDiameter>
-    <torque>20</torque>
-    <commandTopic>/cmd_vel</commandTopic>
-    <odometryTopic>/mobile_robot/odom</odometryTopic>
-    <odometryFrame>odom</odometryFrame>
-    <robotBaseFrame>base_link</robotBaseFrame>
-  </plugin>
 </robot>
